File: Sprite_Sail_60x60cm.brd (EAGLE design)
At the start: 600 x 600 mm, 280 parts

Commit message: Add files via upload
Parts:
- moved L21 1.47 mm to (21.7, 19.5)
- moved C132 1.47 mm to (9.26, 29.0)
- moved R116 1.47 mm to (11.4, 34.6)
- moved L22 1.47 mm to (20.3, 32.4)
- moved R127 1.47 mm to (21.0, 35.1)
- moved U$44 1.47 mm to (12.1, 46.7)
- moved R118 1.47 mm to (20.4, 17.3)
- moved C123 1.47 mm to (24.3, 21.3)
- moved C138 1.47 mm to (23.5, 6.55)
- moved FRONT_PANEL5 1.47 mm to (39.1, 26.3)
- moved L24 1.47 mm to (24.8, 17.1)
- moved LED18 1.47 mm to (25.7, 24.9)
- moved LS12 1.47 mm to (20.5, 16.1)
- moved R111 1.47 mm to (16.6, 13.6)
- moved R119 1.47 mm to (17.2, 32.0)
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Other:
- outline, holes or cut-outs redrawn
- board text added: "1"
- board text added: "2"
- board text added: "3"
- board text added: "4"
- board text removed: "Sprite 1"
- board text removed: "Sprite 2"
- board text removed: "Sprite 3"
- board text removed: "Sprite 4"
